File: money mate.kicad_pcb (KiCad board)
At the start: 2 copper layers, 3.6 x 3.2 mm, 17 parts, among them SW1 SW_Push, SW2 SW_Push, SW3 SW_Push, SW4 RotaryEncoder_Switch, U1 MOUDLE-SEEEDUINO-XIAO

Commit message: pcb ready!!!!
Parts:
- added G***: LOGO, logo:megaLogo, F.Cu at (131.0, 63.5)
- moved SW3 97.6 mm to (191.1, 81.9)
- moved SW4 85.7 mm to (181.8, 56.0)
- moved U2 77.6 mm to (177.4, 64.4), turned to 180 degrees
- moved SW2 73.6 mm to (167.6, 81.9)
- moved SW1 53.6 mm to (144.0, 81.9)
- moved R1 39.1 mm to (102.5, 73.5), turned to 90 degrees
- moved C1 25.2 mm to (117.5, 75.5), turned to -90 degrees
- moved U1 24.5 mm to (112.9, 62.1)
- moved C2 23.9 mm to (117.5, 80.0), turned to -90 degrees
- moved C3 22.2 mm to (117.5, 85.0), turned to -90 degrees
- moved C4 20.5 mm to (117.5, 90.0), turned to -90 degrees
- moved C5 18.8 mm to (117.5, 95.0), turned to -90 degrees
- moved D1 5.70 mm to (109.0, 75.5), turned to 180 degrees
- moved D2 5.70 mm to (109.0, 80.4), turned to 180 degrees
- moved D3 5.70 mm to (109.0, 85.3), turned to 180 degrees
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Connections:
- SW1 pad 1: Net-(U1-PA6_A10_D10_MOSI) -> Net-(U1-PA7_A8_D8_SCK)
- SW3 pad 1: Net-(U1-PA7_A8_D8_SCK) -> Net-(U1-PA6_A10_D10_MOSI)
Routing:
- net GND: track 0.00 -> 215.2 mm, vias 0 -> 10
- net /ROTS1: track 0.00 -> 106.8 mm
- net Net-(U1-PA6_A10_D10_MOSI): track 0.00 -> 97.0 mm
- net /vcc: track 0.00 -> 94.7 mm, vias 0 -> 5
- net /rot_b: track 0.00 -> 89.9 mm
- net /rot_a: track 0.00 -> 83.3 mm
- net Net-(U1-PA5_A9_D9_MISO): track 0.00 -> 82.6 mm
- net Net-(U1-PA7_A8_D8_SCK): track 0.00 -> 59.7 mm
- net Net-(U1-PA8_A4_D4_SDA): track 0.00 -> 53.5 mm
- net Net-(U1-PA9_A5_D5_SCL): track 0.00 -> 50.8 mm
- net Net-(U1-PA11_A3_D3): track 0.00 -> 13.1 mm
- net Net-(D1-DOUT): track 0.00 -> 9.10 mm
- net Net-(D2-DOUT): track 0.00 -> 9.08 mm
- net Net-(D4-DOUT): track 0.00 -> 8.56 mm
- net Net-(D3-DOUT): track 0.00 -> 8.56 mm
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- added copper zone on B.Cu, net GND
Other:
- board size 3.6 x 3.2 mm -> 100 x 50 mm
